File: hardware/slick_bug.kicad_pcb (KiCad board)
At the start: 2 copper layers, 20.2 x 23.1 mm, 10 parts, among them J1 Conn_01x04_Socket, J2 Conn_01x04_Socket, U1 XIAO-RP2040-SMD, U4 MAX40203AUK+T

Commit message: move slick bug stuff to own folder
Parts:
- F1: footprint easyeda:F0805 -> slick_bug:F0805
- J1: footprint halfr:R50_horizontal_4pin -> slick_bug:R50_horizontal_4pin
- J2: footprint halfr:Harwin_M20-89004xx_1x04_P2.54mm_Horizontal_blank -> slick_bug:Harwin_M20-89004xx_1x04_P2.54mm_Horizontal_blank
- U1: footprint Seeed_Studio_XIAO_Series:XIAO-RP2040-SMD -> slick_bug:XIAO-RP2040-SMD
- U2, U3: footprint halfr:R50_pcb_comb -> slick_bug:R50_pcb_comb
- U4: footprint easyeda:SOT-23-5_L3.0-W1.6-P0.95-LS2.8-BR -> slick_bug:SOT-23-5_L3.0-W1.6-P0.95-LS2.8-BR
Changed lines of the file:
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@@
 		)
 	)
-	(footprint "halfr:R50_pcb_comb"
+	(footprint "slick_bug:R50_pcb_comb"
 		(layer "F.Cu")
 		(at 90.75 84.8 180)
@@
 		(embedded_fonts no)
 	)
-	(footprint "halfr:R50_pcb_comb"
+	(footprint "slick_bug:R50_pcb_comb"
 		(layer "F.Cu")
 		(at 90.75 58.1936)
@@
 		(embedded_fonts no)
 	)
-	(footprint "Seeed_Studio_XIAO_Series:XIAO-RP2040-SMD"
+	(footprint "slick_bug:XIAO-RP2040-SMD"
 		(locked yes)
 		(layer "F.Cu")
@@
 		)
 		(embedded_fonts no)
-		(model "${KIPRJMOD}/kicad_assets/halfr.3dshapes/Seeed Studio XIAO RP2040.step"
+		(model "${KIPRJMOD}/lib/slick_bug.3dshapes/Seeed Studio XIAO RP2040.step"
 			(offset
 				(xyz 8.9 10.05 0)
@@
 		)
 	)
-	(footprint "easyeda:SOT-23-5_L3.0-W1.6-P0.95-LS2.8-BR"
+	(footprint "slick_bug:SOT-23-5_L3.0-W1.6-P0.95-LS2.8-BR"
 		(layer "B.Cu")
 		(at 98.5 67.25 180)
@@
 		)
 		(embedded_fonts no)
-		(model "${KIPRJMOD}/kicad_assets/easyeda.3dshapes/SOT-23-5_L3.0-W1.6-P0.95-LS2.8-BR.step"
+		(model "${KIPRJMOD}/lib/slick_bug.3dshapes/SOT-23-5_L3.0-W1.6-P0.95-LS2.8-BR.step"
 			(offset
 				(xyz 0 0 0)
@@
 		)
 	)
-	(footprint "halfr:R50_horizontal_4pin"
+	(footprint "slick_bug:R50_horizontal_4pin"
 		(locked yes)
 		(layer "B.Cu")
@@
 		)
 		(embedded_fonts no)
-		(model "${KIPRJMOD}/kicad_assets/halfr.3dshapes/R50-2C_Main.step"
+		(model "${KIPRJMOD}/lib/slick_bug.3dshapes/R50-2C_Main.step"
 			(offset
 				(xyz -1.9 0.5 0.45)
@@
 			)
 		)
-		(model "${KIPRJMOD}/kicad_assets/halfr.3dshapes/R50-2C_Main.step"
+		(model "${KIPRJMOD}/lib/slick_bug.3dshapes/R50-2C_Main.step"
 			(offset
 				(xyz -0.63 2 0.45)
@@
 			)
 		)
-		(model "${KIPRJMOD}/kicad_assets/halfr.3dshapes/R50-2C_Main.step"
+		(model "${KIPRJMOD}/lib/slick_bug.3dshapes/R50-2C_Main.step"
 			(offset
 				(xyz 0.63 2 0.45)
@@
 			)
 		)
-		(model "${KIPRJMOD}/kicad_assets/halfr.3dshapes/R50-2C_Main.step"
+		(model "${KIPRJMOD}/lib/slick_bug.3dshapes/R50-2C_Main.step"
 			(offset
 				(xyz 1.9 2 0.45)
@@
 			)
 		)
-		(model "${KIPRJMOD}/kicad_assets/halfr.3dshapes/R50_pcb_comb_Main(1).step"
+		(model "${KIPRJMOD}/lib/slick_bug.3dshapes/R50_pcb_comb_Main(1).step"
 			(offset
 				(xyz 29.3 0 -1)
@@
 		)
 	)
-	(footprint "easyeda:F0805"
+	(footprint "slick_bug:F0805"
 		(layer "B.Cu")
 		(at 95 62.25)
@@
 		)
 		(embedded_fonts no)
-		(model "${KIPRJMOD}/kicad_assets/easyeda.3dshapes/F0805_L2.1-W1.4-H0.8.step"
+		(model "${KIPRJMOD}/lib/slick_bug.3dshapes/F0805_L2.1-W1.4-H0.8.step"
 			(offset
 				(xyz 0 0 0)
@@
 		)
 	)
-	(footprint "halfr:Harwin_M20-89004xx_1x04_P2.54mm_Horizontal_blank"
+	(footprint "slick_bug:Harwin_M20-89004xx_1x04_P2.54mm_Horizontal_blank"
 		(locked yes)
 		(layer "B.Cu")
@@
 		)
 		(embedded_fonts no)
-		(model "${LOCAL_ASSETS}/halfr.3dshapes/m20-89004xx_asm.stp"
+		(model "${KIPRJMOD}/lib/slick_bug.3dshapes/m20-89004xx_asm.stp"
 			(offset
 				(xyz 0.5 -6.35 1.5)
